Commit message: fixing inertials- effort controllers

File: lynxbot_description/urdf/arm/link_joint_macro.urdf.xacro (robot description, xacro)
@@ -6,13 +6,7 @@
     radius origin_xyz origin_rpy color_name color mass">
     <link name="${link_name}">
-      <inertial>
-      <mass value="${mass}"/>
-      <origin xyz="0.0 0 0" rpy=" 0 0 0"/>
-      <inertia
-          ixx="0.1" ixy="0" ixz="0"
-          iyy="0.1" iyz="0"
-          izz="0.1"
-      />
-    </inertial>
+      <xacro:cylinder_inertial radius="${radius}" length="${length}" mass="${mass}">
+        <origin xyz="${origin_xyz}" rpy="${origin_rpy}"/>
+      </xacro:cylinder_inertial>
       <visual>
         <geometry>
@@ -26,5 +20,5 @@
       <collision>
         <geometry>
-          <cylinder length="${length}" radius="${radius}"/>
+          <cylinder length="${length*0.5}" radius="${radius*0.5}"/>
         </geometry>
         <origin xyz="${origin_xyz}" rpy="${origin_rpy}"/>
@@ -39,7 +33,7 @@
     <parent link="${parent}"/>
     <axis xyz="${axis_xyz}" rpy="${axis_rpy}"/>
-    <limit effort="30.0" velocity="1.0" lower="${lower_limit}" upper="${upper_limit}"/>
+    <limit effort="100.0" velocity="1.0" lower="${lower_limit}" upper="${upper_limit}"/>
     <joint_properties damping="20.0" friction="10.0"/>
-    <safety_controller k_velocity="10.0" k_position="15.0" soft_lower_limit="${lower_limit}" soft_upper_limit="${upper_limit}" />
+    <!--safety_controller k_velocity="10.0" k_position="15.0" soft_lower_limit="${lower_limit}" soft_upper_limit="${upper_limit}" /-->
   </joint>
   </xacro:macro>
@@ -47,13 +41,7 @@
   origin_xyz origin_rpy color_name color mass">
     <link name="${link_name}">
-      <inertial>
-      <mass value="${mass}"/>
-      <origin xyz="0.0 0 0" rpy=" 0 0 0"/>
-      <inertia
-          ixx="0.1" ixy="0" ixz="0"
-          iyy="0.1" iyz="0"
-          izz="0.1"
-      />
-    </inertial>
+      <xacro:box_inertial x="${size_x}" y="${size_y}" z="${size_z}" m="${mass}">
+        <origin xyz="${origin_xyz}" rpy="${origin_rpy}"/>
+      </xacro:box_inertial>
       <visual>
         <geometry>
@@ -67,5 +55,5 @@
       <collision>
         <geometry>
-          <box size="${size_x} ${size_y} ${size_z}"/>
+          <box size="${size_x*0.5} ${size_y*0.5} ${size_z*0.5}"/>
         </geometry>
         <origin xyz="${origin_xyz}" rpy="${origin_rpy}"/>

File: lynxbot_description/urdf/arm/my_arm.urdf.xacro (robot description, xacro)
@@ -25,5 +25,5 @@
               color_name = "blue"
               color = "0 0 1 1"
-              mass = "0.5"/>
+              mass = "${m_arm_base}"/>
   <arm_link link_name="link_0" length="0.04" radius="0.01"
               origin_xyz="0.045 0 0.02"
@@ -31,5 +31,5 @@
               color_name = "green"
               color = "0 1 0 1"
-              mass = "0.1"/>
+              mass = "${m_0}"/>
   <arm_joint joint_name="joint_0" parent="arm_base" child = "link_0"
                type = "revolute"
@@ -45,5 +45,5 @@
               color_name = "red"
               color = "1 0 0 1"
-              mass = "0.2"/>
+              mass = "${m_1}"/>
   <arm_joint joint_name="joint_1" parent="link_0" child = "link_1"
                type = "revolute"
@@ -59,5 +59,5 @@
               color_name = "green"
               color = "0 0 1 1"
-              mass = "0.2"/>
+              mass = "${m_2}"/>
   <arm_joint joint_name="joint_2" parent="link_1" child = "link_2"
                type = "revolute"
@@ -73,5 +73,5 @@
               color_name = "red"
               color = "1 0 1 1"
-              mass = "0.2"/>
+              mass = "${m_3}"/>
   <arm_joint joint_name="joint_3" parent="link_2" child = "link_3"
                type = "revolute"
@@ -87,5 +87,5 @@
               color_name = "blue"
               color = "0 0 1 1"
-              mass = "0.2"/>
+              mass = "${m_4}"/>
   <arm_joint joint_name="joint_4" parent="link_3" child = "link_4"
                type = "revolute"
@@ -101,5 +101,5 @@
               color_name = "green"
               color = "0 1 0 1"
-              mass = "0.2"/>
+              mass = "${m_5}"/>
   <arm_joint joint_name="joint_5" parent="link_4" child = "link_5"
                type = "revolute"
@@ -117,5 +117,5 @@
               color_name = "green"
               color = "0 1 0 1"
-              mass = "0.2"/>
+              mass = "${m_ee}"/>
   <arm_joint joint_name="joint_ee_base" parent="${parent}" child = "ee_base"
                type = "fixed"
@@ -131,5 +131,5 @@
               color_name = "green"
               color = "0 1 0 1"
-              mass = "0.2"/>
+              mass = "${m_f1}"/>
   <arm_joint joint_name="joint_finger1" parent="ee_base" child = "finger1"
                type = "prismatic"
@@ -145,5 +145,5 @@
               color_name = "green"
               color = "0 1 0 1"
-              mass = "0.2"/>
+              mass = "${m_f2}"/>
   <arm_joint joint_name="joint_finger2" parent="ee_base" child = "finger2"
                type = "prismatic"

File: lynxbot_description/urdf/arm/transmissions.urdf.xacro (robot description, xacro)
@@ -4,9 +4,9 @@
       <type>transmission_interface/SimpleTransmission</type>
       <joint name="joint_0">
-        <hardwareInterface>hardware_interface/PositionJointInterface</hardwareInterface>
+        <hardwareInterface>hardware_interface/EffortJointInterface</hardwareInterface>
       </joint>
       <actuator name="motor_joint_0">
         <mechanicalReduction>1</mechanicalReduction>
-	<hardwareInterface>hardware_interface/PositionJointInterface</hardwareInterface>
+	<hardwareInterface>hardware_interface/EffortJointInterface</hardwareInterface>
       </actuator>
     </transmission>
@@ -14,9 +14,9 @@
       <type>transmission_interface/SimpleTransmission</type>
       <joint name="joint_1">
-        <hardwareInterface>hardware_interface/PositionJointInterface</hardwareInterface>
+        <hardwareInterface>hardware_interface/EffortJointInterface</hardwareInterface>
       </joint>
       <actuator name="motor_joint_1">
         <mechanicalReduction>1</mechanicalReduction>
-	<hardwareInterface>hardware_interface/PositionJointInterface</hardwareInterface>
+	<hardwareInterface>hardware_interface/EffortJointInterface</hardwareInterface>
       </actuator>
     </transmission>
@@ -24,9 +24,9 @@
       <type>transmission_interface/SimpleTransmission</type>
       <joint name="joint_2">
-        <hardwareInterface>hardware_interface/PositionJointInterface</hardwareInterface>
+        <hardwareInterface>hardware_interface/EffortJointInterface</hardwareInterface>
       </joint>
       <actuator name="motor_joint_2">
         <mechanicalReduction>1</mechanicalReduction>
-	<hardwareInterface>hardware_interface/PositionJointInterface</hardwareInterface>
+	<hardwareInterface>hardware_interface/EffortJointInterface</hardwareInterface>
       </actuator>
     </transmission>
@@ -34,9 +34,9 @@
       <type>transmission_interface/SimpleTransmission</type>
       <joint name="joint_3">
-        <hardwareInterface>hardware_interface/PositionJointInterface</hardwareInterface>
+        <hardwareInterface>hardware_interface/EffortJointInterface</hardwareInterface>
       </joint>
       <actuator name="motor_joint_3">
         <mechanicalReduction>1</mechanicalReduction>
-	<hardwareInterface>hardware_interface/PositionJointInterface</hardwareInterface>
+	<hardwareInterface>hardware_interface/EffortJointInterface</hardwareInterface>
       </actuator>
     </transmission>
@@ -44,9 +44,9 @@
       <type>transmission_interface/SimpleTransmission</type>
       <joint name="joint_4">
-        <hardwareInterface>hardware_interface/PositionJointInterface</hardwareInterface>
+        <hardwareInterface>hardware_interface/EffortJointInterface</hardwareInterface>
       </joint>
       <actuator name="motor_joint_4">
         <mechanicalReduction>1</mechanicalReduction>
-	<hardwareInterface>hardware_interface/PositionJointInterface</hardwareInterface>
+	<hardwareInterface>hardware_interface/EffortJointInterface</hardwareInterface>
       </actuator>
     </transmission>
@@ -54,9 +54,9 @@
       <type>transmission_interface/SimpleTransmission</type>
       <joint name="joint_5">
-        <hardwareInterface>hardware_interface/PositionJointInterface</hardwareInterface>
+        <hardwareInterface>hardware_interface/EffortJointInterface</hardwareInterface>
       </joint>
       <actuator name="motor_joint_5">
         <mechanicalReduction>1</mechanicalReduction>
-	<hardwareInterface>hardware_interface/PositionJointInterface</hardwareInterface>
+	<hardwareInterface>hardware_interface/EffortJointInterface</hardwareInterface>
       </actuator>
     </transmission>
@@ -64,9 +64,9 @@
       <type>transmission_interface/SimpleTransmission</type>
       <joint name="joint_finger1">
-        <hardwareInterface>hardware_interface/PositionJointInterface</hardwareInterface>
+        <hardwareInterface>hardware_interface/EffortJointInterface</hardwareInterface>
       </joint>
       <actuator name="motor_joint_finger1">
         <mechanicalReduction>1</mechanicalReduction>
-	<hardwareInterface>hardware_interface/PositionJointInterface</hardwareInterface>
+	<hardwareInterface>hardware_interface/EffortJointInterface</hardwareInterface>
       </actuator>
     </transmission>
@@ -74,9 +74,9 @@
       <type>transmission_interface/SimpleTransmission</type>
       <joint name="joint_finger2">
-        <hardwareInterface>hardware_interface/PositionJointInterface</hardwareInterface>
+        <hardwareInterface>hardware_interface/EffortJointInterface</hardwareInterface>
       </joint>
       <actuator name="motor_joint_finger2">
         <mechanicalReduction>1</mechanicalReduction>
-	<hardwareInterface>hardware_interface/PositionJointInterface</hardwareInterface>
+	<hardwareInterface>hardware_interface/EffortJointInterface</hardwareInterface>
       </actuator>
     </transmission>

File: lynxbot_description/urdf/common_properties.urdf.xacro (robot description, xacro)
@@ -25,5 +25,5 @@
   <xacro:property name="lidar_base_joint_z" value="0.0275" />
   <xacro:property name="ydlidar_tilt" value="${M_PI/2 + (-2.5)*(M_PI/180)}" />
-  <xacro:property name="ydlidar_joint_z" value="0.015" />
+  <xacro:property name="ydlidar_joint_z" value="0.025" />
   <!-- kinect base-->
   <xacro:property name="kinect_base1_height" value="0.38" />
@@ -35,5 +35,5 @@
   <xacro:property name="cam_px" value="0.03" />
   <xacro:property name="cam_py" value="0.0" />
-  <xacro:property name="cam_pz" value="0.06" />
+  <xacro:property name="cam_pz" value="0.09" />
   <xacro:property name="cam_or" value="0.0" />
   <xacro:property name="cam_op" value="0.2" />
@@ -45,3 +45,13 @@
   <xacro:property name="arm_parent" value="wood_base" />
   <xacro:property name="ee_parent" value="link_5" />
+  <xacro:property name="m_arm_base" value="0.4" />
+  <xacro:property name="m_0" value="0.3" />
+  <xacro:property name="m_1" value="0.4" />
+  <xacro:property name="m_2" value="0.8" />
+  <xacro:property name="m_3" value="0.1" />
+  <xacro:property name="m_4" value="0.1" />
+  <xacro:property name="m_5" value="0.1" />
+  <xacro:property name="m_ee" value="0.1" />
+  <xacro:property name="m_f1" value="0.03" />
+  <xacro:property name="m_f2" value="0.03" />
 </robot>

File: lynxbot_description/urdf/lynx_rover.urdf.xacro (robot description, xacro)
@@ -8,4 +8,5 @@
   <xacro:include filename="$(find lynxbot_description)/urdf/transmissions.urdf.xacro" />
   <xacro:include filename="$(find lynxbot_description)/urdf/sensors/kinect.urdf.xacro" />
+  <xacro:include filename="$(find lynxbot_description)/urdf/macros/inertia_macros.urdf.xacro" />
   <!--xacro:include filename="$(find lynxbot_description)/urdf/macros/inertia_macros.urdf.xacro" /-->
   <xacro:arg name="sim" default="false"/>
@@ -22,14 +23,7 @@
   </joint>
   <link name='chassis'>
-    <pose>0 0 0 0 0 0</pose>
-    <inertial>
-      <mass value="5.0"/>
-      <origin xyz="0.0 0 0" rpy=" 0 0 0"/>
-      <inertia
-          ixx="0.1" ixy="0" ixz="0"
-          iyy="0.1" iyz="0"
-          izz="0.1"
-      />
-    </inertial>
+      <xacro:box_inertial x="${Length_base}" y="${Width_base}" z="${Height_base}" m="500">
+        <origin xyz="0 0 0" rpy="0 0 0"/>
+      </xacro:box_inertial>
     <collision name='collision'>
       <origin xyz="0 0 0" rpy=" 0 0 0"/>

File: lynxbot_description/urdf/macros/inertia_macros.urdf.xacro (robot description, xacro)
@@ -12,5 +12,5 @@
   <xacro:macro name="box_inertial" params="x y z m *origin">
     <inertial>
-      <mass value="${mass}" />
+      <mass value="${m}" />
       <xacro:insert_block name="origin" />
       <inertia  ixx="${m*(y*y+z*z)/12}" ixy = "0" ixz = "0"

File: lynxbot_description/urdf/macros/wheels.urdf.xacro (robot description, xacro)
@@ -4,13 +4,7 @@
   <xacro:macro name="wheel_link" params="prefix origin_xyz origin_rpy">
     <link name="${prefix}_wheel">
-      <inertial>
-        <mass value="5"/>
+      <xacro:cylinder_inertial radius="0.055" length="0.065" mass="5">
         <origin xyz="${origin_xyz}" rpy="${origin_rpy}"/>
-        <inertia
-          ixx="0.1" ixy="0" ixz="0"
-          iyy="0.1" iyz="0"
-          izz="0.1"
-          />
-       </inertial>
+      </xacro:cylinder_inertial>
       <visual>
         <geometry>
@@ -24,5 +18,5 @@
       <collision>
         <geometry>
-          <cylinder length="0.065" radius="0.055"/>
+          <cylinder length="0.03" radius="0.05"/>
         </geometry>
         <origin xyz="${origin_xyz}" rpy="${origin_rpy}"/>
@@ -37,5 +31,5 @@
     <axis xyz="0 1 0" rpy="0 0 0"/>
     <limit effort="10000" velocity="1000"/>
-    <joint_properties damping="1.0" friction="1.0"/>
+    <joint_properties damping="20.0" friction="10.0"/>
   </joint>
   </xacro:macro>

File: lynxbot_description/urdf/object.urdf.xacro (robot description, xacro)
@@ -1,12 +1,11 @@
 <?xml version='1.0'?>
 <robot name="simple_box" xmlns:xacro="http://www.ros.org/wiki/xacro">
+  <xacro:include filename="$(find lynxbot_description)/urdf/macros/inertia_macros.urdf.xacro" />
   <link name="my_box">
-    <inertial>
-      <origin xyz="2 0.5 0" />
-      <mass value="0.1" />
-      <inertia  ixx="1.0" ixy="0.0"  ixz="0.0"  iyy="100.0"  iyz="0.0"  izz="1.0" />
-    </inertial>
+      <xacro:box_inertial x="0.04" y="0.04" z="0.07" m="0.1">
+        <origin xyz="2.0 0.0 0.0" rpy="0 0 0"/>
+      </xacro:box_inertial>
     <visual>
-      <origin xyz="2 0 1"/>
+      <origin xyz="2 0 0"/>
       <geometry>
         <box size="0.04 0.04 0.07" />
@@ -14,5 +13,5 @@
     </visual>
     <collision>
-      <origin xyz="2 0 1"/>
+      <origin xyz="2 0 0"/>
       <geometry>
         <box size="0.04 0.04 0.07" />

File: lynxbot_description/urdf/sensor_bases.urdf.xacro (robot description, xacro)
@@ -5,10 +5,10 @@
     <link name="wood_base">
       <inertial>
-        <mass value="0.1"/>
+        <mass value="0.01"/>
         <origin xyz="0 0 0" rpy="0 0 0"/>
         <inertia
-          ixx="0.1" ixy="0" ixz="0"
-          iyy="0.1" iyz="0"
-          izz="0.1"
+          ixx="0.00001" ixy="0" ixz="0"
+          iyy="0.00001" iyz="0"
+          izz="0.00001"
         />
       </inertial>
@@ -38,10 +38,10 @@
     <link name="lidar_base">
       <inertial>
-        <mass value="0.1"/>
+        <mass value="0.01"/>
         <origin xyz="0 0 0" rpy="0 0 0"/>
         <inertia
-          ixx="0.1" ixy="0" ixz="0"
-          iyy="0.1" iyz="0"
-          izz="0.1"
+          ixx="0.0001" ixy="0" ixz="0"
+          iyy="0.0001" iyz="0"
+          izz="0.0001"
         />
       </inertial>
@@ -72,10 +72,10 @@
     <link name="kinect_base1">
       <inertial>
-        <mass value="0.1"/>
+        <mass value="0.01"/>
         <origin xyz="0 0 0" rpy="0 0 0"/>
         <inertia
-          ixx="0.1" ixy="0" ixz="0"
-          iyy="0.1" iyz="0"
-          izz="0.1"
+          ixx="0.000001" ixy="0" ixz="0"
+          iyy="0.000001" iyz="0"
+          izz="0.000001"
         />
       </inertial>
@@ -106,10 +106,10 @@
     <link name="kinect_base2">
       <inertial>
-        <mass value="0.1"/>
+        <mass value="0.01"/>
         <origin xyz="0 0 0" rpy="0 0 0"/>
         <inertia
-          ixx="0.1" ixy="0" ixz="0"
-          iyy="0.1" iyz="0"
-          izz="0.1"
+          ixx="0.000001" ixy="0" ixz="0"
+          iyy="0.00001" iyz="0"
+          izz="0.00001"
         />
       </inertial>

File: lynxbot_description/urdf/sensors/ydlidar.urdf.xacro (robot description, xacro)
@@ -29,5 +29,5 @@
     <origin xyz="0 0 ${ydlidar_joint_z}" rpy="0 0 ${ydlidar_tilt}"/>
     <child link="laser_frame"/>
-    <parent link="lidar_base"/>
+    <parent link="chassis"/>
   </joint>
 </robot>
