Commit message: Fixed simulation

File: lynxbot_description/urdf/arm/link_joint_macro.urdf.xacro (robot description, xacro)
@@ -34,5 +34,5 @@
     <axis xyz="${axis_xyz}" rpy="${axis_rpy}"/>
     <limit effort="100.0" velocity="1.0" lower="${lower_limit}" upper="${upper_limit}"/>
-    <joint_properties damping="20.0" friction="10.0"/>
+    <joint_properties damping="0.0" friction="10.0"/>
     <!--safety_controller k_velocity="10.0" k_position="15.0" soft_lower_limit="${lower_limit}" soft_upper_limit="${upper_limit}" /-->
   </joint>

File: lynxbot_description/urdf/arm/transmissions.urdf.xacro (robot description, xacro)
@@ -4,9 +4,9 @@
       <type>transmission_interface/SimpleTransmission</type>
       <joint name="joint_0">
-        <hardwareInterface>hardware_interface/EffortJointInterface</hardwareInterface>
+        <hardwareInterface>hardware_interface/PositionJointInterface</hardwareInterface>
       </joint>
       <actuator name="motor_joint_0">
         <mechanicalReduction>1</mechanicalReduction>
-	<hardwareInterface>hardware_interface/EffortJointInterface</hardwareInterface>
+	<hardwareInterface>hardware_interface/PositionJointInterface</hardwareInterface>
       </actuator>
     </transmission>
@@ -14,9 +14,9 @@
       <type>transmission_interface/SimpleTransmission</type>
       <joint name="joint_1">
-        <hardwareInterface>hardware_interface/EffortJointInterface</hardwareInterface>
+        <hardwareInterface>hardware_interface/PositionJointInterface</hardwareInterface>
       </joint>
       <actuator name="motor_joint_1">
         <mechanicalReduction>1</mechanicalReduction>
-	<hardwareInterface>hardware_interface/EffortJointInterface</hardwareInterface>
+	<hardwareInterface>hardware_interface/PositionJointInterface</hardwareInterface>
       </actuator>
     </transmission>
@@ -24,9 +24,9 @@
       <type>transmission_interface/SimpleTransmission</type>
       <joint name="joint_2">
-        <hardwareInterface>hardware_interface/EffortJointInterface</hardwareInterface>
+        <hardwareInterface>hardware_interface/PositionJointInterface</hardwareInterface>
       </joint>
       <actuator name="motor_joint_2">
         <mechanicalReduction>1</mechanicalReduction>
-	<hardwareInterface>hardware_interface/EffortJointInterface</hardwareInterface>
+	<hardwareInterface>hardware_interface/PositionJointInterface</hardwareInterface>
       </actuator>
     </transmission>
@@ -34,9 +34,9 @@
       <type>transmission_interface/SimpleTransmission</type>
       <joint name="joint_3">
-        <hardwareInterface>hardware_interface/EffortJointInterface</hardwareInterface>
+        <hardwareInterface>hardware_interface/PositionJointInterface</hardwareInterface>
       </joint>
       <actuator name="motor_joint_3">
         <mechanicalReduction>1</mechanicalReduction>
-	<hardwareInterface>hardware_interface/EffortJointInterface</hardwareInterface>
+	<hardwareInterface>hardware_interface/PositionJointInterface</hardwareInterface>
       </actuator>
     </transmission>
@@ -44,9 +44,9 @@
       <type>transmission_interface/SimpleTransmission</type>
       <joint name="joint_4">
-        <hardwareInterface>hardware_interface/EffortJointInterface</hardwareInterface>
+        <hardwareInterface>hardware_interface/PositionJointInterface</hardwareInterface>
       </joint>
       <actuator name="motor_joint_4">
         <mechanicalReduction>1</mechanicalReduction>
-	<hardwareInterface>hardware_interface/EffortJointInterface</hardwareInterface>
+	<hardwareInterface>hardware_interface/PositionJointInterface</hardwareInterface>
       </actuator>
     </transmission>
@@ -54,9 +54,9 @@
       <type>transmission_interface/SimpleTransmission</type>
       <joint name="joint_5">
-        <hardwareInterface>hardware_interface/EffortJointInterface</hardwareInterface>
+        <hardwareInterface>hardware_interface/PositionJointInterface</hardwareInterface>
       </joint>
       <actuator name="motor_joint_5">
         <mechanicalReduction>1</mechanicalReduction>
-	<hardwareInterface>hardware_interface/EffortJointInterface</hardwareInterface>
+	<hardwareInterface>hardware_interface/PositionJointInterface</hardwareInterface>
       </actuator>
     </transmission>
@@ -64,9 +64,9 @@
       <type>transmission_interface/SimpleTransmission</type>
       <joint name="joint_finger1">
-        <hardwareInterface>hardware_interface/EffortJointInterface</hardwareInterface>
+        <hardwareInterface>hardware_interface/PositionJointInterface</hardwareInterface>
       </joint>
       <actuator name="motor_joint_finger1">
         <mechanicalReduction>1</mechanicalReduction>
-	<hardwareInterface>hardware_interface/EffortJointInterface</hardwareInterface>
+	<hardwareInterface>hardware_interface/PositionJointInterface</hardwareInterface>
       </actuator>
     </transmission>
@@ -74,9 +74,9 @@
       <type>transmission_interface/SimpleTransmission</type>
       <joint name="joint_finger2">
-        <hardwareInterface>hardware_interface/EffortJointInterface</hardwareInterface>
+        <hardwareInterface>hardware_interface/PositionJointInterface</hardwareInterface>
       </joint>
       <actuator name="motor_joint_finger2">
         <mechanicalReduction>1</mechanicalReduction>
-	<hardwareInterface>hardware_interface/EffortJointInterface</hardwareInterface>
+	<hardwareInterface>hardware_interface/PositionJointInterface</hardwareInterface>
       </actuator>
     </transmission>

File: lynxbot_description/urdf/common_properties.urdf.xacro (robot description, xacro)
@@ -25,5 +25,5 @@
   <xacro:property name="lidar_base_joint_z" value="0.0275" />
   <xacro:property name="ydlidar_tilt" value="${M_PI/2 + (-2.5)*(M_PI/180)}" />
-  <xacro:property name="ydlidar_joint_z" value="0.025" />
+  <xacro:property name="ydlidar_joint_z" value="0.055" />
   <!-- kinect base-->
   <xacro:property name="kinect_base1_height" value="0.38" />
@@ -45,11 +45,11 @@
   <xacro:property name="arm_parent" value="wood_base" />
   <xacro:property name="ee_parent" value="link_5" />
-  <xacro:property name="m_arm_base" value="0.4" />
-  <xacro:property name="m_0" value="0.3" />
-  <xacro:property name="m_1" value="0.4" />
-  <xacro:property name="m_2" value="0.8" />
-  <xacro:property name="m_3" value="0.1" />
-  <xacro:property name="m_4" value="0.1" />
-  <xacro:property name="m_5" value="0.1" />
+  <xacro:property name="m_arm_base" value="100" />
+  <xacro:property name="m_0" value="0.01" />
+  <xacro:property name="m_1" value="0.01" />
+  <xacro:property name="m_2" value="0.01" />
+  <xacro:property name="m_3" value="0.01" />
+  <xacro:property name="m_4" value="0.01" />
+  <xacro:property name="m_5" value="0.01" />
   <xacro:property name="m_ee" value="0.1" />
   <xacro:property name="m_f1" value="0.03" />

File: lynxbot_description/urdf/lynx_rover.urdf.xacro (robot description, xacro)
@@ -23,7 +23,9 @@
   </joint>
   <link name='chassis'>
-      <xacro:box_inertial x="${Length_base}" y="${Width_base}" z="${Height_base}" m="500">
-        <origin xyz="0 0 0" rpy="0 0 0"/>
-      </xacro:box_inertial>
+   <inertial>
+     <origin xyz="0 0 0" rpy="0 0 0"/>
+     <mass value="100"/>
+     <inertia ixx="0.5"  ixy="0"  ixz="0" iyy="0.5" iyz="0" izz="0.5" />
+   </inertial>
     <collision name='collision'>
       <origin xyz="0 0 0" rpy=" 0 0 0"/>

File: lynxbot_description/urdf/macros/inertia_macros.urdf.xacro (robot description, xacro)
@@ -1,5 +1,5 @@
 <?xml version="1.0" ?>
 <robot name="my_robot_arm" xmlns:xacro="http://www.ros.org/wiki/xacro">
-  <xacro:macro name="cylinder_inertial" params="radius length mass *origin">
+  <!--xacro:macro name="cylinder_inertial" params="radius length mass *origin">
     <inertial>
       <mass value="${mass}" />
@@ -18,4 +18,22 @@
                   izz="${m*(x*x+z*z)/12}" />
     </inertial>
+  </xacro:macro-->
+  <xacro:macro name="cylinder_inertial" params="radius length mass *origin">
+    <inertial>
+      <mass value="${mass}" />
+      <xacro:insert_block name="origin" />
+      <inertia  ixx="0.0001" ixy = "0" ixz = "0"
+                  iyy="0.0001" iyz = "0"
+                  izz="0.0001" />
+    </inertial>
+  </xacro:macro>
+  <xacro:macro name="box_inertial" params="x y z m *origin">
+    <inertial>
+      <mass value="${m}" />
+      <xacro:insert_block name="origin" />
+      <inertia  ixx="0.0001" ixy = "0" ixz = "0"
+                  iyy="0.0001" iyz = "0"
+                  izz="0.0001" />
+    </inertial>
   </xacro:macro>
 </robot>

File: lynxbot_description/urdf/macros/wheels.urdf.xacro (robot description, xacro)
@@ -4,7 +4,9 @@
   <xacro:macro name="wheel_link" params="prefix origin_xyz origin_rpy">
     <link name="${prefix}_wheel">
-      <xacro:cylinder_inertial radius="0.055" length="0.065" mass="5">
-        <origin xyz="${origin_xyz}" rpy="${origin_rpy}"/>
-      </xacro:cylinder_inertial>
+   <inertial>
+     <origin xyz="0 0 0" rpy="0 0 0"/>
+     <mass value="100"/>
+     <inertia ixx="0.15"  ixy="0"  ixz="0" iyy="0.15" iyz="0" izz="0.15" />
+   </inertial>
       <visual>
         <geometry>
@@ -18,5 +20,5 @@
       <collision>
         <geometry>
-          <cylinder length="0.03" radius="0.05"/>
+          <cylinder length="0.065" radius="0.055"/>
         </geometry>
         <origin xyz="${origin_xyz}" rpy="${origin_rpy}"/>

File: lynxbot_description/urdf/sensor_bases.urdf.xacro (robot description, xacro)
@@ -35,5 +35,5 @@
     </joint>
   </xacro:macro>
-  <xacro:macro name="lidar_base">
+  <!--xacro:macro name="lidar_base">
     <link name="lidar_base">
       <inertial>
@@ -61,12 +61,12 @@
         <origin xyz="0 0 0.005" rpy="0 0 0"/>
       </collision>
-    </link>
+    </link-->
     <!-- -0.057 from center of the robot wood base 0.0575 forward so -11.45 from wood center-->
-    <joint name="lidar_base_joint" type="fixed">
+    <!--joint name="lidar_base_joint" type="fixed">
       <origin xyz="${lidar_base_joint_x} ${lidar_base_joint_y} ${lidar_base_joint_z}" rpy="0 0 0" />
       <parent link="chassis"/>
       <child link="lidar_base" />
     </joint>
-  </xacro:macro>
+  </xacro:macro-->
   <xacro:macro name="kinect_base1">
     <link name="kinect_base1">
@@ -75,7 +75,7 @@
         <origin xyz="0 0 0" rpy="0 0 0"/>
         <inertia
-          ixx="0.000001" ixy="0" ixz="0"
-          iyy="0.000001" iyz="0"
-          izz="0.000001"
+          ixx="0.0001" ixy="0" ixz="0"
+          iyy="0.0001" iyz="0"
+          izz="0.0001"
         />
       </inertial>
@@ -109,7 +109,7 @@
         <origin xyz="0 0 0" rpy="0 0 0"/>
         <inertia
-          ixx="0.000001" ixy="0" ixz="0"
-          iyy="0.00001" iyz="0"
-          izz="0.00001"
+          ixx="0.0001" ixy="0" ixz="0"
+          iyy="0.0001" iyz="0"
+          izz="0.0001"
         />
       </inertial>

File: lynxbot_description/urdf/sensors/ydlidar.urdf.xacro (robot description, xacro)
@@ -6,5 +6,5 @@
     <inertial>
       <mass value="0.1"/>
-      <origin xyz="0 0 0" rpy="0 0 0"/>
+      <origin xyz="0 0 0.0" rpy="0 0 0"/>
       <inertia
           ixx="1e-6" ixy="0" ixz="0"
