Commit message: fixing up

File: lynxbot_description/urdf/common_properties.urdf.xacro (robot description, xacro)
@@ -17,11 +17,5 @@
   <xacro:property name="wood_joint_y" value="0.0" />
   <xacro:property name="wood_joint_z" value="0.1275" />
-  <!-- lidar base-->
-  <xacro:property name="lidar_base_size_x" value="0.04" />
-  <xacro:property name="lidar_base_size_y" value="0.07" />
-  <xacro:property name="lidar_base_size_z" value="0.01" />
-  <xacro:property name="lidar_base_joint_x" value="0.015" />
-  <xacro:property name="lidar_base_joint_y" value="0.0" />
-  <xacro:property name="lidar_base_joint_z" value="0.0275" />
+  <!-- lidar -->
   <xacro:property name="ydlidar_tilt" value="${M_PI/2 + (-2.5)*(M_PI/180)}" />
   <xacro:property name="ydlidar_joint_z" value="0.055" />

Commit message: smaller wheels

File: lynxbot_description/urdf/common_properties.urdf.xacro (robot description, xacro)
@@ -16,20 +16,21 @@
   <xacro:property name="wood_joint_x" value="0.05" />
   <xacro:property name="wood_joint_y" value="0.0" />
-  <xacro:property name="wood_joint_z" value="0.1275" />
+  <xacro:property name="wood_joint_z" value="0.115" />
   <!-- lidar -->
-  <xacro:property name="ydlidar_tilt" value="${M_PI/2 + (-2.5)*(M_PI/180)}" />
-  <xacro:property name="ydlidar_joint_z" value="0.055" />
+  <xacro:property name="ydlidar_tilt" value="${M_PI + (-1.25)*(M_PI/180)}" />
+  <xacro:property name="ydlidar_joint_z" value="0.035" />
+  <xacro:property name="ydlidar_joint_x" value="0.025" />
   <!-- kinect base-->
   <xacro:property name="kinect_base1_height" value="0.38" />
   <xacro:property name="kinect_base2_joint_z" value="0.18" />
+  <xacro:property name="kinect_base1_joint_z" value="0.2" />
   <xacro:property name="kinect_base1_joint_x" value="-0.14" />
   <xacro:property name="kinect_base1_joint_y" value="0.0" />
-  <xacro:property name="kinect_base1_joint_z" value="0.2" />
   <xacro:property name="kinect_parent" value="kinect_base2" />
-  <xacro:property name="cam_px" value="0.03" />
+  <xacro:property name="cam_px" value="0.02" />
   <xacro:property name="cam_py" value="0.0" />
-  <xacro:property name="cam_pz" value="0.09" />
+  <xacro:property name="cam_pz" value="0.06" />
   <xacro:property name="cam_or" value="0.0" />
-  <xacro:property name="cam_op" value="0.2" />
+  <xacro:property name="cam_op" value="0.0" />
   <xacro:property name="cam_oy" value="0.0" />
   <!-- Arm -->

File: lynxbot_description/urdf/macros/wheels.urdf.xacro (robot description, xacro)
@@ -11,5 +11,5 @@
       <visual>
         <geometry>
-          <cylinder length="0.065" radius="0.055"/>
+          <cylinder length="0.065" radius="0.03"/>
         </geometry>
         <origin xyz="${origin_xyz}" rpy="${origin_rpy}"/>
@@ -20,5 +20,5 @@
       <collision>
         <geometry>
-          <cylinder length="0.065" radius="0.055"/>
+          <cylinder length="0.065" radius="0.03"/>
         </geometry>
         <origin xyz="${origin_xyz}" rpy="${origin_rpy}"/>

File: lynxbot_description/urdf/sensors/ydlidar.urdf.xacro (robot description, xacro)
@@ -27,5 +27,5 @@
   </link>
   <joint type="fixed" name="ydlidar_joint">
-    <origin xyz="0 0 ${ydlidar_joint_z}" rpy="0 0 ${ydlidar_tilt}"/>
+    <origin xyz="${ydlidar_joint_x} 0 ${ydlidar_joint_z}" rpy="0 0 ${ydlidar_tilt}"/>
     <child link="laser_frame"/>
     <parent link="chassis"/>

Commit message: making class cpp

File: lynxbot_description/urdf/common_properties.urdf.xacro (robot description, xacro)
@@ -18,15 +18,15 @@
   <xacro:property name="wood_joint_z" value="0.115" />
   <!-- lidar -->
-  <xacro:property name="ydlidar_tilt" value="${M_PI + (-1.25)*(M_PI/180)}" />
+  <xacro:property name="ydlidar_tilt" value="${M_PI + (-3.5)*(M_PI/180)}" />
   <xacro:property name="ydlidar_joint_z" value="0.035" />
-  <xacro:property name="ydlidar_joint_x" value="0.025" />
+  <xacro:property name="ydlidar_joint_x" value="0.026" />
   <!-- kinect base-->
   <xacro:property name="kinect_base1_height" value="0.38" />
   <xacro:property name="kinect_base2_joint_z" value="0.18" />
   <xacro:property name="kinect_base1_joint_z" value="0.2" />
-  <xacro:property name="kinect_base1_joint_x" value="-0.14" />
+  <xacro:property name="kinect_base1_joint_x" value="-0.10" />
   <xacro:property name="kinect_base1_joint_y" value="0.0" />
   <xacro:property name="kinect_parent" value="kinect_base2" />
-  <xacro:property name="cam_px" value="0.02" />
+  <xacro:property name="cam_px" value="0.03" />
   <xacro:property name="cam_py" value="0.0" />
   <xacro:property name="cam_pz" value="0.06" />
